Commit message: Lidar-link non-zero inertia

File: src/gazebo_differential_drive_robot/urdf/robot.urdf (robot description, URDF)
Before this commit: robot differential_drive_robot, 6 links, 5 joints
Links:
- link lidar_link: mass 1e-6 -> 0.0001

File: src/gazebo_differential_drive_robot/urdf/robot.xacro (robot description, xacro)
@@ -144,6 +144,6 @@
         </collision>
         <inertial>
-            <mass value="1e-6"/>
-            <inertia ixx="1e-6" ixy="0.0" ixz="0.0" iyy="1e-6" iyz="0" izz="1e-6"/>
+            <mass value="0.0001"/>
+            <inertia ixx="0.0001" ixy="0.0" ixz="0.0" iyy="0.0001" iyz="0" izz="0.0001"/>
             <origin xyz="0 0 0" rpy="0 0 0"/>
         </inertial>

Commit message: Added camera support

File: src/gazebo_differential_drive_robot/urdf/robot.urdf (robot description, URDF)
Before this commit: robot differential_drive_robot, 6 links, 5 joints
Links:
- added link camera_link; visual box size=0.025 0.05 0.05
- added link camera_link_optical
Joints:
- added joint camera_joint: type fixed, parent base_link, child camera_link, origin xyz=0.15 0 0.0125 rpy=0 0 0
- added joint camera_optical_joint: type fixed, parent camera_link, child camera_link_optical, origin xyz=0 0 0 rpy=-1.5707963267948966 0 -1.5707963267948966
- joint lidar_joint: origin xyz=0.049999999999999996 0 0.05 rpy=0 0 0 -> xyz=0 0 0.05 rpy=0 0 0

File: src/gazebo_differential_drive_robot/urdf/robot.xacro (robot description, xacro)
@@ -149,4 +149,15 @@
         </inertial>
     </link>
+    <link name="camera_link">
+        <visual>
+            <geometry>
+                <box size="0.025 0.05 0.05"/>
+            </geometry>
+            <material name="camera_material">
+                <color rgba="1.0 0.0 0.0 1.0"/>
+            </material>
+        </visual>
+    </link>
+    <link name="camera_link_optical"></link>
     <!-- Joints -->
     <!-- Base Link Joint -->
@@ -182,8 +193,18 @@
     <!-- Lidar Joint (fixed) -->
     <joint name="lidar_joint" type="fixed">
-        <origin xyz="${caster_offset/2} 0 ${lidar_width}" rpy="0 0 0"/>
+        <origin xyz="0 0 ${lidar_width}" rpy="0 0 0"/>
         <parent link="base_link"/>
         <child link="lidar_link"/>
         <axis xyz="0 1 0" rpt="0 0 0" />
+    </joint>
+    <joint name="camera_joint" type="fixed">
+        <parent link="base_link"/>
+        <child link="camera_link"/>
+        <origin xyz="${body_length/2} 0 ${body_height/8}" rpy="0 0 0"/>
+    </joint>
+    <joint name="camera_optical_joint" type="fixed">
+        <parent link="camera_link"/>
+        <child link="camera_link_optical"/>
+        <origin xyz="0 0 0" rpy="${-pi/2} 0 ${-pi/2}"/>
     </joint>
     <!-- Gazebo Parameters -->
@@ -205,4 +226,5 @@
     </gazebo>
     <!-- Gazebo plugins -->
+    <!--
     <gazebo>
         <plugin filename="gz-sim-diff-drive-system" name="gz::sim::systems::DiffDrive">
@@ -227,4 +249,5 @@
         </plugin>
     </gazebo>
+    -->
     <gazebo reference="lidar_link">
         <!-- Required: 'gpu_ray' is optimized for Harmonic/Ogre2 -->
@@ -269,4 +292,25 @@
         </sensor>
     </gazebo>
+    <gazebo reference="camera_link">
+        <sensor name="camera" type="camera">
+            <pose> 0 0 0 0 0 0 </pose>
+            <visualize>true</visualize>
+            <update_rate>10</update_rate>
+            <camera>
+                <horizontal_fov>1.089</horizontal_fov>
+                <image>
+                    <format>R8G8B8</format>
+                    <width>640</width>
+                    <height>480</height>
+                </image>
+                <clip>
+                    <near>0.05</near>
+                    <far>8.0</far>
+                </clip>
+            </camera>
+            <topic>camera/image_raw</topic>
+            <gz_frame_id>camera_link_optical</gz_frame_id>
+        </sensor>
+    </gazebo>
     <ros2_control name="GazeboSimSystem" type="system">
         <hardware>

Commit message: Still trying to load imu sensor

File: src/gazebo_differential_drive_robot/urdf/robot.urdf (robot description, URDF)
Before this commit: robot differential_drive_robot, 8 links, 7 joints
Links:
- added link imu_link, mass 0.0001; visual box size=0.05 0.05 0.02
- link camera_link: mass None -> 0.0001
Joints:
- added joint imu_joint: type fixed, parent base_link, child imu_link, origin xyz=-0.11499999999999999 0 0.05 rpy=0 0 0

File: src/gazebo_differential_drive_robot/urdf/robot.xacro (robot description, xacro)
@@ -158,6 +158,26 @@
             </material>
         </visual>
+        <inertial>
+            <mass value="0.0001"/>
+            <inertia ixx="0.0001" ixy="0.0" ixz="0.0" iyy="0.0001" iyz="0" izz="0.0001"/>
+            <origin xyz="0 0 0" rpy="0 0 0"/>
+        </inertial>
     </link>
     <link name="camera_link_optical"></link>
+    <link name="imu_link">
+        <visual>
+            <geometry>
+                <box size="0.05 0.05 0.02"/>
+            </geometry>
+            <material name="imu_material">
+                <color rgba="0.0 1.0 1.0 1.0"/>
+            </material>
+        </visual>
+        <inertial>
+            <mass value="0.0001"/>
+            <inertia ixx="0.0001" ixy="0.0" ixz="0.0" iyy="0.0001" iyz="0" izz="0.0001"/>
+            <origin xyz="0 0 0" rpy="0 0 0"/>
+        </inertial>
+    </link>
     <!-- Joints -->
     <!-- Base Link Joint -->
@@ -208,4 +228,9 @@
         <origin xyz="0 0 0" rpy="${-pi/2} 0 ${-pi/2}"/>
     </joint>
+    <joint name="imu_joint" type="fixed">
+        <parent link="base_link"/>
+        <child link="imu_link"/>
+        <origin xyz="${-body_length/4 - 0.04} 0 ${body_height/2}" rpy="0 0 0"/>
+    </joint>
     <!-- Gazebo Parameters -->
     <gazebo reference="base_link">
@@ -222,4 +247,12 @@
     </gazebo>
     <gazebo reference="caster_link">
+        <mu1>0.000001</mu1>
+        <mu2>0.000001</mu2>
+    </gazebo>
+    <gazebo reference="camera_link">
+        <mu1>0.000001</mu1>
+        <mu2>0.000001</mu2>
+    </gazebo>
+    <gazebo reference="imu_link">
         <mu1>0.000001</mu1>
         <mu2>0.000001</mu2>
@@ -313,4 +346,12 @@
         </sensor>
     </gazebo>
+    <gazebo reference="imu_link">
+        <sensor name="imu_sensor" type="imu">
+            <always_on>true</always_on>
+            <update_rate>100</update_rate>
+            <visualize>true</visualize>
+            <topic>imu</topic>
+        </sensor>
+    </gazebo>
     <ros2_control name="GazeboSimSystem" type="system">
         <hardware>
@@ -327,4 +368,16 @@
             <state_interface name="velocity"/>
         </joint>
+        <sensor name="imu_sensor">
+            <state_interface name="orientation.x"/>
+            <state_interface name="orientation.y"/>
+            <state_interface name="orientation.z"/>
+            <state_interface name="orientation.w"/>
+            <state_interface name="angular_velocity.x"/>
+            <state_interface name="angular_velocity.y"/>
+            <state_interface name="angular_velocity.z"/>
+            <state_interface name="linear_acceleration.x"/>
+            <state_interface name="linear_acceleration.y"/>
+            <state_interface name="linear_acceleration.z"/>
+        </sensor>
     </ros2_control>
     <gazebo>
@@ -332,4 +385,7 @@
             <parameters>$(find gazebo_differential_drive_robot)/config/ros2_controllers.yaml</parameters>
         </plugin>
+        <plugin filename="gz-sim-imu-system" name="gz::sim::systems::Imu">
+            <parameters>$(find gazebo_differential_drive_robot)/config/ros2_controllers.yaml</parameters>
+        </plugin>
     </gazebo>
 </robot>
