Commit message: Added ros2_control

File: src/gazebo_differential_drive_robot/urdf/robot.xacro (robot description, xacro)
@@ -187,4 +187,19 @@
         <axis xyz="0 1 0" rpt="0 0 0" />
     </joint>
+  <ros2_control name="GazeboSimSystem" type="system">
+    <hardware>
+      <plugin>gz_ros2_control/GazeboSimSystem</plugin>
+    </hardware>
+    <joint name="left_wheel_joint">
+      <command_interface name="velocity"/>
+      <state_interface name="position"/>
+      <state_interface name="velocity"/>
+    </joint>
+    <joint name="right_wheel_joint">
+      <command_interface name="velocity"/>
+      <state_interface name="position"/>
+      <state_interface name="velocity"/>
+    </joint>
+  </ros2_control>
     <!-- Gazebo Parameters -->
     <gazebo reference="base_link">
@@ -264,5 +279,4 @@
         </noise>
       </ray>
-      <!-- Harmonic uses the combined gz-sim-sensors-system plugin -->
       <plugin filename="gz-sim-sensors-system" name="gz::sim::systems::Sensors">
         <render_type>ogre2</render_type>
@@ -270,3 +284,10 @@
     </sensor>
   </gazebo>
+<!--
+  <gazebo>
+    <plugin filename="gz_ros2_control-system" name="gz_ros2_control::GazeboSimROS2ControlPlugin">
+      <parameters>$(find gazebo_differential_drive_robot)/config/ros2_controllers.yaml</parameters>
+    </plugin>
+  </gazebo>
+-->
 </robot>

Commit message: Re-arrange gazebo plugins

File: src/gazebo_differential_drive_robot/urdf/robot.xacro (robot description, xacro)
@@ -187,19 +187,4 @@
         <axis xyz="0 1 0" rpt="0 0 0" />
     </joint>
-  <ros2_control name="GazeboSimSystem" type="system">
-    <hardware>
-      <plugin>gz_ros2_control/GazeboSimSystem</plugin>
-    </hardware>
-    <joint name="left_wheel_joint">
-      <command_interface name="velocity"/>
-      <state_interface name="position"/>
-      <state_interface name="velocity"/>
-    </joint>
-    <joint name="right_wheel_joint">
-      <command_interface name="velocity"/>
-      <state_interface name="position"/>
-      <state_interface name="velocity"/>
-    </joint>
-  </ros2_control>
     <!-- Gazebo Parameters -->
     <gazebo reference="base_link">
@@ -219,5 +204,5 @@
         <mu2>0.000001</mu2>
     </gazebo>
-    <!-- Gazebo Plugins -->
+    <!-- Gazebo plugins -->
     <gazebo>
         <plugin filename="gz-sim-diff-drive-system" name="gz::sim::systems::DiffDrive">
@@ -242,50 +227,65 @@
         </plugin>
     </gazebo>
-  <gazebo reference="lidar_link">
-    <!-- Required: 'gpu_ray' is optimized for Harmonic/Ogre2 -->
-    <sensor name="lidar_link" type="gpu_ray">
-      <pose relative_to='lidar_link'>0 0 ${lidar_width/2} 0 0 0</pose>
-      <topic>/scan</topic>
-      <gz_frame_id>lidar_link</gz_frame_id>
-      <update_rate>10.0</update_rate>
-      <always_on>1</always_on>
-      <visualize>true</visualize>
-      <ray>
-        <scan>
-          <horizontal>
-            <samples>360</samples>
-            <resolution>1</resolution>
-            <min_angle>-3.14159</min_angle>
-            <max_angle>3.14159</max_angle>
-          </horizontal>
-          <!-- Explicitly force a single vertical slice for 2D operation -->
-          <vertical>
-            <samples>1</samples>
-            <resolution>1</resolution>
-            <min_angle>0.0</min_angle>
-            <max_angle>0.0</max_angle>
-          </vertical>
-        </scan>
-        <range>
-          <min>0.12</min>
-          <max>12.0</max>
-          <resolution>0.01</resolution>
-        </range>
-        <!-- Optional noise modeling mimicking real-world data -->
-        <noise>
-          <type>gaussian</type>
-          <mean>0.0</mean>
-          <stddev>0.01</stddev>
-        </noise>
-      </ray>
-      <plugin filename="gz-sim-sensors-system" name="gz::sim::systems::Sensors">
-        <render_type>ogre2</render_type>
-      </plugin>
-    </sensor>
-  </gazebo>
-  <gazebo>
-    <plugin filename="gz_ros2_control-system" name="gz_ros2_control::GazeboSimROS2ControlPlugin">
-      <parameters>$(find gazebo_differential_drive_robot)/config/ros2_controllers.yaml</parameters>
-    </plugin>
-  </gazebo>
+    <gazebo reference="lidar_link">
+        <!-- Required: 'gpu_ray' is optimized for Harmonic/Ogre2 -->
+        <sensor name="lidar_link" type="gpu_ray">
+        <pose relative_to='lidar_link'>0 0 ${lidar_width/2} 0 0 0</pose>
+        <topic>/scan</topic>
+        <gz_frame_id>lidar_link</gz_frame_id>
+        <update_rate>10.0</update_rate>
+        <always_on>1</always_on>
+        <visualize>true</visualize>
+        <ray>
+            <scan>
+            <horizontal>
+                <samples>360</samples>
+                <resolution>1</resolution>
+                <min_angle>-3.14159</min_angle>
+                <max_angle>3.14159</max_angle>
+            </horizontal>
+            <!-- Explicitly force a single vertical slice for 2D operation -->
+            <vertical>
+                <samples>1</samples>
+                <resolution>1</resolution>
+                <min_angle>0.0</min_angle>
+                <max_angle>0.0</max_angle>
+            </vertical>
+            </scan>
+            <range>
+            <min>0.12</min>
+            <max>12.0</max>
+            <resolution>0.01</resolution>
+            </range>
+            <!-- Optional noise modeling mimicking real-world data -->
+            <noise>
+            <type>gaussian</type>
+            <mean>0.0</mean>
+            <stddev>0.01</stddev>
+            </noise>
+        </ray>
+        <plugin filename="gz-sim-sensors-system" name="gz::sim::systems::Sensors">
+            <render_type>ogre2</render_type>
+        </plugin>
+        </sensor>
+    </gazebo>
+    <ros2_control name="GazeboSimSystem" type="system">
+        <hardware>
+            <plugin>gz_ros2_control/GazeboSimSystem</plugin>
+        </hardware>
+        <joint name="left_wheel_joint">
+            <command_interface name="velocity"/>
+            <state_interface name="position"/>
+            <state_interface name="velocity"/>
+        </joint>
+        <joint name="right_wheel_joint">
+            <command_interface name="velocity"/>
+            <state_interface name="position"/>
+            <state_interface name="velocity"/>
+        </joint>
+    </ros2_control>
+    <gazebo>
+        <plugin filename="gz_ros2_control-system" name="gz_ros2_control::GazeboSimROS2ControlPlugin">
+        <parameters>$(find gazebo_differential_drive_robot)/config/ros2_controllers.yaml</parameters>
+        </plugin>
+    </gazebo>
 </robot>

Commit message: First pass at an arm

File: src/gazebo_differential_drive_robot/urdf/robot.xacro (robot description, xacro)
@@ -233,4 +233,5 @@
         <origin xyz="${-body_length/4 - 0.04} 0 ${body_height/2}" rpy="0 0 0"/>
     </joint>
+    <xacro:include filename="arm.xacro" />
     <!-- Gazebo Parameters -->
     <gazebo reference="base_link">
@@ -381,4 +382,40 @@
             <state_interface name="linear_acceleration.z"/>
         </sensor>
+        <joint name="joint_1">
+            <command_interface name="position">
+                <param name="min">-3.14</param>
+                <param name="max">3.14</param>
+            </command_interface>
+            <state_interface name="position">
+                <param name="initial_value">0.0</param>
+            </state_interface>
+            <state_interface name="velocity"/>
+        </joint>
+        <joint name="joint_2">
+            <command_interface name="position">
+                <param name="min">-1.57</param>
+                <param name="max">1.57</param>
+            </command_interface>
+            <state_interface name="position">
+                <param name="initial_value">0.0</param>
+            </state_interface>
+            <state_interface name="velocity"/>
+        </joint>
+        <joint name="left_finger_joint">
+            <command_interface name="position">
+                <param name="min">0.0</param>
+                <param name="max">0.04</param>
+            </command_interface>
+            <state_interface name="position">
+                <param name="initial_value">0.0</param>
+            </state_interface>
+            <state_interface name="velocity"/>
+        </joint>
+        <joint name="right_finger_joint">
+             <state_interface name="position">
+                <param name="initial_value">0.0</param>
+            </state_interface>
+            <state_interface name="velocity"/>
+        </joint>
     </ros2_control>
     <gazebo>
@@ -386,4 +423,4 @@
             <parameters>$(find gazebo_differential_drive_robot)/config/ros2_controllers.yaml</parameters>
         </plugin>
-     </gazebo>
+    </gazebo>
 </robot>

Commit message: Re-run moveit assistant

File: src/gazebo_differential_drive_robot/urdf/robot.xacro (robot description, xacro)
@@ -158,4 +158,9 @@
             </material>
         </visual>
+        <collision>
+            <geometry>
+                <box size="0.025 0.05 0.05"/>
+            </geometry>
+        </collision>
         <inertial>
             <mass value="0.0001"/>
@@ -174,4 +179,9 @@
             </material>
         </visual>
+        <collision>
+            <geometry>
+                <box size="0.05 0.05 0.02"/>
+            </geometry>
+        </collision>
         <inertial>
             <mass value="0.0001"/>
