Commit message: Re-do moveit assistant again

File: src/gazebo_differential_drive_robot/urdf/arm.xacro (robot description, xacro)
@@ -3,4 +3,9 @@
   <!-- ==================== Arm Links & Joints ==================== -->
   <xacro:property name="arm_offset" value="${body_length/2 - caster_radius}"/>
+  <joint name="virtual_joint" type="planar">
+    <command_interface name="position"/>
+    <state_interface name="position"/>
+    <state_interface name="velocity"/>
+  </joint>
   <!-- Shoulder Joint (Rotation around Z) -->
   <joint name="joint_1" type="revolute">

Commit message: Still working on moveit :(

File: src/gazebo_differential_drive_robot/urdf/arm.xacro (robot description, xacro)
@@ -3,9 +3,6 @@
   <!-- ==================== Arm Links & Joints ==================== -->
   <xacro:property name="arm_offset" value="${body_length/2 - caster_radius}"/>
-  <joint name="virtual_joint" type="planar">
-    <command_interface name="position"/>
-    <state_interface name="position"/>
-    <state_interface name="velocity"/>
-  </joint>
+  <!-- Virtual Joint -->
+  <virtual_joint name="virtual_joint" type="planar" parent_frame="odom" child_link="base_footprint" />
   <!-- Shoulder Joint (Rotation around Z) -->
   <joint name="joint_1" type="revolute">
@@ -85,5 +82,5 @@
   <!-- ==================== Gripper Fingers ==================== -->
   <!-- Left Finger (Prismatic Active Joint) -->
-<!-- The main active joint controlled by the gripper plugin -->
+  <!-- The main active joint controlled by the gripper plugin -->
   <joint name="left_finger_joint" type="prismatic">
     <parent link="gripper_base"/>

File: src/gazebo_differential_drive_robot/urdf/robot.xacro (robot description, xacro)
@@ -370,4 +370,9 @@
             <plugin>gz_ros2_control/GazeboSimSystem</plugin>
         </hardware>
+        <joint name="virtual_joint">
+            <command_interface name="position"/>
+            <state_interface name="position"/>
+            <state_interface name="velocity"/>
+        </joint>
         <joint name="left_wheel_joint">
             <command_interface name="velocity"/>

Commit message: Remove moveit directory

File: src/gazebo_differential_drive_robot/urdf/arm.xacro (robot description, xacro)
@@ -3,6 +3,4 @@
   <!-- ==================== Arm Links & Joints ==================== -->
   <xacro:property name="arm_offset" value="${body_length/2 - caster_radius}"/>
-  <!-- Virtual Joint -->
-  <virtual_joint name="virtual_joint" type="planar" parent_frame="odom" child_link="base_footprint" />
   <!-- Shoulder Joint (Rotation around Z) -->
   <joint name="joint_1" type="revolute">

File: src/gazebo_differential_drive_robot/urdf/robot.xacro (robot description, xacro)
@@ -370,9 +370,4 @@
             <plugin>gz_ros2_control/GazeboSimSystem</plugin>
         </hardware>
-        <joint name="virtual_joint">
-            <command_interface name="position"/>
-            <state_interface name="position"/>
-            <state_interface name="velocity"/>
-        </joint>
         <joint name="left_wheel_joint">
             <command_interface name="velocity"/>
