Commit message: Moveit is still a mess

File: src/moveit_differential_drive_robot/config/differential_drive_robot.ros2_control.xacro (robot description, xacro)
@@ -29,11 +29,4 @@
                 <state_interface name="velocity"/>
             </joint>
-            <joint name="virtual_joint">
-                <command_interface name="position"/>
-                <state_interface name="position">
-                  <param name="initial_value">${initial_positions['virtual_joint']}</param>
-                </state_interface>
-                <state_interface name="velocity"/>
-            </joint>
         </ros2_control>
     </xacro:macro>
